File: Hardware/BipolarCircuit.kicad_sch (KiCad schematic)
At the start: 24 parts, among them U1 MCP4822, U2 X_OPAMP, U3 -X_OPAMP, U4 Y_OPAMP, U5 -X_OPAMP

Commit message: Revised the circuit diagram
Parts:
- removed A1: Arduino_UNO_R3, Module:Arduino_UNO_R3, symbol MCU_Module:Arduino_UNO_R3
- added U?: Logic Level Shifter, Package_SO:TSSOP-20_4.4x6.5mm_P0.65mm, symbol Logic_LevelTranslator:TXS0108EPW
- added XA?: Arduino_Due_Shield, symbol arduino:Arduino_Due_Shield
Connections:
- net 5V_ARDUINO: now also U1.1 (Vdd), U?.10 (OE), U?.19 (VCCB), XA?.5V1 (5V)
- net GND: now also XA?.GND1 (GND)
- net GROUND: now also U?.11 (GND)
- net CS_5V: now reaches U1.2 (~{CS})
- net CS_5V: now also U?.20 (B1)
- net MOSI_5V: now reaches U1.4 (SDI)
- net MOSI_5V: now also U?.17 (B3)
- net SCK_5V: now reaches U1.3 (SCK)
- net SCK_5V: now also U?.18 (B2)
- new net 3V3_ARDUINO: U?.2 (VCCA), XA?.3V3 (3.3V)
- new net CS_3V3: U?.1 (A1), XA?.D10 (D10_CS0)
- new net LASER_SWITCH_3V3: U?.5 (A4), XA?.D8
- new net LASER_SWITCH_5V: U?.16 (B4)
- new net MOSI_3V3: U?.4 (A3), XA?.MOSI (SPI_MOSI)
- new net SCK_3V3: U?.3 (A2), XA?.SCK (SPI_SCK)
