File: Hardware/BipolarCircuit.sch (KiCad schematic (older format))
At the start: 24 parts, among them U1 MCP4822, U2 X_OPAMP, U3 -X_OPAMP, U4 Y_OPAMP, U5 -X_OPAMP

Commit message: Fixed the context menu of the canvas, if a background picture was loaded in
Parts:
- R11, R14: value 221 -> 2k
Changed lines of the file:
@@
 P 6850 950
 F 0 "R11" V 7057 950 50  0001 C CNN
-F 1 "221" V 6965 950 50  0000 C CNN
+F 1 "2k" V 6965 950 50  0000 C CNN
 F 2 "" V 6780 950 50  0001 C CNN
 F 3 "~" H 6850 950 50  0001 C CNN
@@
 P 7550 950
 F 0 "R14" V 7757 950 50  0001 C CNN
-F 1 "221" V 7665 950 50  0000 C CNN
+F 1 "2k" V 7665 950 50  0000 C CNN
 F 2 "" V 7480 950 50  0001 C CNN
 F 3 "~" H 7550 950 50  0001 C CNN

Commit message: Revised the code to work with the Arduino Due
Parts:
- removed A1: Arduino_UNO_R3, Module:Arduino_UNO_R3, symbol MCU_Module:Arduino_UNO_R3
- removed U1: MCP4822, symbol Analog_DAC:MCP4822
- added U?: Logic Level Shifter, Package_DFN_QFN:WQFN-20-1EP_2.5x4.5mm_P0.5mm_EP1x2.9mm, symbol Logic_LevelTranslator:FXMA108
- added XA?: Arduino_Due_Shield, symbol arduino:Arduino_Due_Shield
Connections:
- net labels added: 3V3_ARDUINO, LASER_SWITCH_3V3, LASER_SWITCH_5V
- net labels removed: GROUND
- wire segments 92 -> 80
